Commit message: Added seperate joints URDF to understand diff types of joints.

File: URDF_practice/joints.urdf (robot description, URDF)
Before this commit: robot success_practice_bot, 3 links, 2 joints
Links:
- removed link third_link
Joints:
- removed joint second_third_joint
- joint base_second_joint: axis (none) -> 1 0 0; limit (none) -> lower=-0.15 upper=0.15 effort=10 velocity=1.0; type fixed -> prismatic
