Commit message: added left wheel

File: RedCherryBot/model.urdf (robot description, URDF)
Before this commit: robot Red_Cherry_Bot, 2 links, 1 joints
Links:
- added link left_wheel_link; visual cylinder length=0.05 radius=0.1
Joints:
- added joint base_left_wheel_joint: type continuous, parent base_link, child left_wheel_link, origin xyz=-0.15 0.225 0 rpy=0 0 0, axis 0 1 0

Commit message: Put Base Footprint link and adjusted offsets.

File: RedCherryBot/model.urdf (robot description, URDF)
Before this commit: robot Red_Cherry_Bot, 3 links, 2 joints
Links:
- added link base_footprint_link
- added link caster_wheel_link; visual sphere radius=0.05
Joints:
- added joint base_caster_wheel_joint: type fixed, parent base_link, child caster_wheel_link, origin xyz=0.2 0 -0.05 rpy=0 0 0
- added joint base_joint: type fixed, parent base_footprint_link, child base_link, origin xyz=0 0 0.1 rpy=0 0 0
