Commit message: Done: xacro renames and some xacro props to avoid hardcoding in the urdf.

File: ros2_ws/src/red_cherrybot_description/urdf/model.urdf.xacro (robot description, xacro)
@@ -1,4 +1,9 @@
 <?xml version="1.0"?>
-<robot name="Red_Cherry_Bot">
+<robot name="Red_Cherry_Bot" xmlns:xacro="http://www.ros.org/wiki/xacro">
+<xacro:property name="base_length" value="0.6"/>
+<xacro:property name="base_width" value="0.4"/>
+<xacro:property name="base_height" value="0.2"/>
+<xacro:property name="wheel_radius" value="0.1"/>
+<xacro:property name="wheel_length" value="0.05"/>
      <!-- Vibrant & Metallic Material Palette -->
 <material name="cherry_light_red">
@@ -13,7 +18,7 @@
     <visual>
       <geometry>
-        <box size="0.6 0.4 0.2"/>
+        <box size="${base_length} ${base_width} ${base_height}"/>
       </geometry>
-      <origin xyz="0 0 0.1" rpy="0 0 0"/>
+      <origin xyz="0 0 ${base_height/2.0}" rpy="0 0 0"/>
       <material name="cherry_light_red"/>
     </visual>
@@ -22,7 +27,7 @@
     <visual>
         <geometry>
-            <cylinder radius="0.1" length="0.05"/>
+            <cylinder radius="${wheel_radius}" length="${wheel_length}"/>
         </geometry>
-        <origin xyz="0 0 0" rpy="1.57 0 0"/>
+        <origin xyz="0 0 0" rpy="${pi/2} 0 0"/>
         <material name="metallic_grey"/>
     </visual>
@@ -31,7 +36,7 @@
     <visual>
         <geometry>
-            <cylinder radius="0.1" length="0.05"/>
+            <cylinder radius="${wheel_radius}" length="${wheel_length}"/>
         </geometry>
-        <origin xyz="0 0 0" rpy="1.57 0 0"/>
+        <origin xyz="0 0 0" rpy="${pi/2} 0 0"/>
         <material name="metallic_grey"/>
     </visual>
@@ -40,5 +45,5 @@
     <visual>
       <geometry>
-        <sphere radius="0.05"/>
+        <sphere radius="${wheel_radius/2.0}"/>
       </geometry>
       <origin xyz="0 0 0" rpy="0 0 0"/>
@@ -53,10 +58,10 @@
   <parent link="base_footprint_link"/>
   <child link="base_link"/>
-  <origin xyz="0 0 0.1" rpy="0 0 0"/> <!-- 0.1 because thats wheel offset from ground, the wheel radius ! We want this joint/TF at the ground ! the base_footprint is the projection of the base on the ground and robot is correctly placed herein ! As base link offset by 0.1, every children of it got by same and nothing actually changes for the parts of the robot.-->
+  <origin xyz="0 0 ${wheel_radius}" rpy="0 0 0"/> <!-- 0.1 because thats wheel offset from ground, the wheel radius ! We want this joint/TF at the ground ! the base_footprint is the projection of the base on the ground and robot is correctly placed herein ! As base link offset by 0.1, every children of it got by same and nothing actually changes for the parts of the robot.-->
 </joint>
   <joint name="base_right_wheel_joint" type="continuous">
     <parent link="base_link"/>
     <child link="right_wheel_link"/>
-    <origin xyz="-0.15 -0.225 0" rpy="0 0 0"/>
+    <origin xyz="-${base_length/4.0} -{base_width/2.0 + wheel_length/2.0} 0" rpy="0 0 0"/>
     <axis xyz="0 1 0"/>
   </joint>
@@ -64,5 +69,5 @@
     <parent link="base_link"/>
     <child link="left_wheel_link"/>
-    <origin xyz="-0.15 0.225 0" rpy="0 0 0"/>
+    <origin xyz="-${base_length/4.0} {base_width/2.0 + wheel_length/2.0} 0" rpy="0 0 0"/>
     <axis xyz="0 1 0"/>
   </joint>
@@ -70,5 +75,5 @@
     <parent link="base_link"/>
     <child link="caster_wheel_link"/>
-    <origin xyz="0.2 0 -0.05" rpy="0 0 0"/>
+    <origin xyz="${base_length/3.0} 0 -0.05" rpy="0 0 0"/>
   </joint>
 </robot>

Commit message: Feat: xacro props used everywhere in urdf, no more hardcoded values. Scaling Up/Down of robot wrt to the prop values work. TRICKY but once we define the props/vars first, it gets easier. :)

File: ros2_ws/src/red_cherrybot_description/urdf/model.urdf.xacro (robot description, xacro)
@@ -1,9 +1,9 @@
 <?xml version="1.0"?>
 <robot name="Red_Cherry_Bot" xmlns:xacro="http://www.ros.org/wiki/xacro">
-<xacro:property name="base_length" value="0.6"/>
-<xacro:property name="base_width" value="0.4"/>
-<xacro:property name="base_height" value="0.2"/>
-<xacro:property name="wheel_radius" value="0.1"/>
-<xacro:property name="wheel_length" value="0.05"/>
+<xacro:property name="base_length" value="1.2"/>
+<xacro:property name="base_width" value="0.8"/>
+<xacro:property name="base_height" value="0.4"/>
+<xacro:property name="wheel_radius" value="0.2"/>
+<xacro:property name="wheel_length" value="0.1"/>
      <!-- Vibrant & Metallic Material Palette -->
 <material name="cherry_light_red">
@@ -63,5 +63,5 @@
     <parent link="base_link"/>
     <child link="right_wheel_link"/>
-    <origin xyz="-${base_length/4.0} -{base_width/2.0 + wheel_length/2.0} 0" rpy="0 0 0"/>
+    <origin xyz="-${base_length/4.0} -${base_width/2.0 + wheel_length/2.0} 0" rpy="0 0 0"/>
     <axis xyz="0 1 0"/>
   </joint>
@@ -69,5 +69,5 @@
     <parent link="base_link"/>
     <child link="left_wheel_link"/>
-    <origin xyz="-${base_length/4.0} {base_width/2.0 + wheel_length/2.0} 0" rpy="0 0 0"/>
+    <origin xyz="-${base_length/4.0} ${base_width/2.0 + wheel_length/2.0} 0" rpy="0 0 0"/>
     <axis xyz="0 1 0"/>
   </joint>
@@ -75,5 +75,5 @@
     <parent link="base_link"/>
     <child link="caster_wheel_link"/>
-    <origin xyz="${base_length/3.0} 0 -0.05" rpy="0 0 0"/>
+    <origin xyz="${base_length/3.0} 0 -${wheel_radius/2.0}" rpy="0 0 0"/>
   </joint>
 </robot>

Commit message: Added XACRO Macros for the 2 wheels (with prefixes).

File: ros2_ws/src/red_cherrybot_description/urdf/model.urdf.xacro (robot description, xacro)
@@ -24,22 +24,18 @@
     </visual>
   </link>
-  <link name="right_wheel_link">
-    <visual>
-        <geometry>
-            <cylinder radius="${wheel_radius}" length="${wheel_length}"/>
-        </geometry>
-        <origin xyz="0 0 0" rpy="${pi/2} 0 0"/>
-        <material name="metallic_grey"/>
-    </visual>
-  </link>
-  <link name="left_wheel_link">
-    <visual>
-        <geometry>
-            <cylinder radius="${wheel_radius}" length="${wheel_length}"/>
-        </geometry>
-        <origin xyz="0 0 0" rpy="${pi/2} 0 0"/>
-        <material name="metallic_grey"/>
-    </visual>
-  </link>
+  <!-- Creating macros for 2 wheels, but before creating a macro think once it makes sense or not to make a macro for it ! Dont Overoptimize and dont create unnecessary complexity ! -->
+  <xacro:macro name="wheel_link" params="prefix">
+    <link name="${prefix}_wheel_link">
+      <visual>
+            <geometry>
+                <cylinder radius="${wheel_radius}" length="${wheel_length}"/>
+            </geometry>
+            <origin xyz="0 0 0" rpy="${pi/2} 0 0"/>
+            <material name="metallic_grey"/>
+      </visual>
+    </link>
+  </xacro:macro>
+  <xacro:wheel_link prefix="right"/>
+  <xacro:wheel_link prefix="left"/>
   <link name="caster_wheel_link">
     <visual>

Commit message: Refactor: separate common properties and mobile base into distinct XACRO files

File: ros2_ws/src/red_cherrybot_description/urdf/model.urdf.xacro (robot description, xacro)
@@ -1,75 +1,5 @@
 <?xml version="1.0"?>
 <robot name="Red_Cherry_Bot" xmlns:xacro="http://www.ros.org/wiki/xacro">
-<xacro:property name="base_length" value="1.2"/>
-<xacro:property name="base_width" value="0.8"/>
-<xacro:property name="base_height" value="0.4"/>
-<xacro:property name="wheel_radius" value="0.2"/>
-<xacro:property name="wheel_length" value="0.1"/>
-     <!-- Vibrant & Metallic Material Palette -->
-<material name="cherry_light_red">
-  <!-- Bright, vibrant cherry red with high saturation -->
-  <color rgba="0.85 0.09 0.21 1.0" />
-</material>
-<material name="metallic_grey">
-  <!-- Mid-tone gunmetal/silver grey finish -->
-  <color rgba="1 1 1 1.0"/>
-</material>
-  <link name="base_link">
-    <visual>
-      <geometry>
-        <box size="${base_length} ${base_width} ${base_height}"/>
-      </geometry>
-      <origin xyz="0 0 ${base_height/2.0}" rpy="0 0 0"/>
-      <material name="cherry_light_red"/>
-    </visual>
-  </link>
-  <!-- Creating macros for 2 wheels, but before creating a macro think once it makes sense or not to make a macro for it ! Dont Overoptimize and dont create unnecessary complexity ! -->
-  <xacro:macro name="wheel_link" params="prefix">
-    <link name="${prefix}_wheel_link">
-      <visual>
-            <geometry>
-                <cylinder radius="${wheel_radius}" length="${wheel_length}"/>
-            </geometry>
-            <origin xyz="0 0 0" rpy="${pi/2} 0 0"/>
-            <material name="metallic_grey"/>
-      </visual>
-    </link>
-  </xacro:macro>
-  <xacro:wheel_link prefix="right"/>
-  <xacro:wheel_link prefix="left"/>
-  <link name="caster_wheel_link">
-    <visual>
-      <geometry>
-        <sphere radius="${wheel_radius/2.0}"/>
-      </geometry>
-      <origin xyz="0 0 0" rpy="0 0 0"/>
-      <material name="metallic_grey"/>
-    </visual>
-  </link>
-  <link name="base_footprint_link">
-    <!--No visual-->
-  </link>
- <!-- We chose to keep visual at 000, joint is centered at the visual. So we added 0.025 to the y-coordinate of cylinder. Why 0.025 ? half of cylinder height. Note that if we put origin = "0 0.025 0" in visual, it would look same, but the structure is a lot different ! And how did we find position of joint ? By halving box lengths, simple but effective. Remianing was the sync the joint with the visual. We did this by ensuring the joint origin matched the visual origin. We DID NOT Edited visual origin this time !-->
-<joint name="base_joint" type="fixed">
-  <parent link="base_footprint_link"/>
-  <child link="base_link"/>
-  <origin xyz="0 0 ${wheel_radius}" rpy="0 0 0"/> <!-- 0.1 because thats wheel offset from ground, the wheel radius ! We want this joint/TF at the ground ! the base_footprint is the projection of the base on the ground and robot is correctly placed herein ! As base link offset by 0.1, every children of it got by same and nothing actually changes for the parts of the robot.-->
-</joint>
-  <joint name="base_right_wheel_joint" type="continuous">
-    <parent link="base_link"/>
-    <child link="right_wheel_link"/>
-    <origin xyz="-${base_length/4.0} -${base_width/2.0 + wheel_length/2.0} 0" rpy="0 0 0"/>
-    <axis xyz="0 1 0"/>
-  </joint>
-  <joint name="base_left_wheel_joint" type="continuous">
-    <parent link="base_link"/>
-    <child link="left_wheel_link"/>
-    <origin xyz="-${base_length/4.0} ${base_width/2.0 + wheel_length/2.0} 0" rpy="0 0 0"/>
-    <axis xyz="0 1 0"/>
-  </joint>
-<joint name="base_caster_wheel_joint" type="fixed">
-    <parent link="base_link"/>
-    <child link="caster_wheel_link"/>
-    <origin xyz="${base_length/3.0} 0 -${wheel_radius/2.0}" rpy="0 0 0"/>
-  </joint>
+<xacro:include filename="common_properties.xacro"/>
+<xacro:include filename="mobile_base.xacro"/>
 </robot>
