Commit message: Completion :) - OpenCV compatibily added using a virtual link in camera.xacro, Z Pointing forward. Persistent camera view removed from urdf config for rviz.

File: ros2_ws/src/red_cherrybot_description/urdf/camera.xacro (robot description, xacro)
@@ -27,4 +27,11 @@
     <origin xyz="${(base_length + camera_length)/2.0} 0 ${base_height/2.0}" rpy="0 0 0"/>
   </joint>
+  <!-- Virtual Link for OpenCV integration -->
+  <link name="camera_link_optical" />
+  <joint name="camera_optical_joint" type="fixed">
+    <parent link="camera_link"/>
+    <child link="camera_link_optical"/>
+    <origin xyz="0 0 0" rpy="${-pi/2.0} 0 ${-pi/2.0}"/>
+  </joint>
   <gazebo reference="camera_link">
     <sensor name="front_camera_sensor" type="camera">
@@ -45,4 +52,5 @@
           <stddev>0.007</stddev>
         </noise>
+        <optical_frame_id>camera_link_optical</optical_frame_id>
         <!-- Camera information topic -->
         <camera_info_topic>camera/camera_info</camera_info_topic>
