Commit message: Feat: add box_inertia macro and apply it to mobile base for realistic mass properties

File: ros2_ws/src/red_cherrybot_description/urdf/common_properties.xacro (robot description, xacro)
@@ -8,5 +8,15 @@
     <material name="bright_white">
         <!-- Bright White finish -->
-        <color rgba="0 0 1 1.0"/>
+        <color rgba="1 1 1 1.0"/>
     </material>
+    <xacro:macro name="box_inertia" params="m x y z o_xyz o_rpy">
+        <inertial>
+               <mass value="${m}"/>
+               <origin xyz="${o_xyz}" rpy="${o_rpy}"/>
+               <inertia
+                    ixx="${ (m/12.0) * (y*y + z*z) }" ixy="0" ixz="0"
+                    iyy="${ (m/12.0) * (x*x + z*z) }" iyz="0"
+                    izz="${ (m/12.0) * (x*x + y*y) }"/>
+        </inertial>
+    </xacro:macro>
 </robot>

File: ros2_ws/src/red_cherrybot_description/urdf/mobile_base.xacro (robot description, xacro)
@@ -14,4 +14,6 @@
       <material name="cherry_light_red"/>
     </visual>
+    <xacro:box_inertia m="10" x="${base_length}" y="${base_width}" z="${base_height}" o_xyz="0 0 ${base_height/2.0}" o_rpy="0 0 0"/>
+    <!-- mass is in KG, so put realistic values though its Simulation. Here its 10Kg -->
   </link>
   <!-- Creating macros for 2 wheels, but before creating a macro think once it makes sense or not to make a macro for it ! Dont Overoptimize and dont create unnecessary complexity ! -->
@@ -39,5 +41,5 @@
   </link>
   <link name="base_footprint_link">
-    <!--No visual-->
+    <!--No visual, or inertia-->
   </link>
  <!-- We chose to keep visual at 000, joint is centered at the visual. So we added 0.025 to the y-coordinate of cylinder. Why 0.025 ? half of cylinder height. Note that if we put origin = "0 0.025 0" in visual, it would look same, but the structure is a lot different ! And how did we find position of joint ? By halving box lengths, simple but effective. Remianing was the sync the joint with the visual. We did this by ensuring the joint origin matched the visual origin. We DID NOT Edited visual origin this time !-->

File: ros2_ws/src/red_cherrybot_description/urdf/model.urdf.xacro (robot description, xacro)
@@ -3,4 +3,4 @@
 <xacro:include filename="common_properties.xacro"/>
 <xacro:include filename="mobile_base.xacro"/>
-<!-- Method to use custom meshes designed in CAD Sfotwares: Create a meshes folder in the pkg, install the folder in CMakeLists.txt and then reference them in the URDF file. Use the mesh include filename syntax. Including the custom mesh in the URDF here is not difficult, but designing it is the actual hard part. We also need to Scale Down/Up frequently in urdf as original STL file of CAD is bigger/smaller.-->
+<!-- Method to use custom meshes designed in CAD Softwares: Create a meshes folder in the pkg, install the folder in CMakeLists.txt and then reference them in the URDF file. Use the mesh include filename syntax. Including the custom mesh in the URDF here is not difficult, but designing it is the actual hard part. We also need to Scale Down/Up frequently in urdf as original STL file of CAD is bigger/smaller.-->
 </robot>

Commit message: Feat: add wheel_inertia (for main side wheels) macro for calculating wheel inertial properties and integrate it into mobile base

File: ros2_ws/src/red_cherrybot_description/urdf/common_properties.xacro (robot description, xacro)
@@ -20,3 +20,13 @@
         </inertial>
     </xacro:macro>
+    <xacro:macro name="wheel_inertia" params="m r l o_xyz o_rpy">
+        <inertial>
+            <mass value="${m}"/>
+            <origin xyz="${o_xyz}" rpy="${o_rpy}"/>
+            <inertia
+                ixx="${ (m/12.0) * (3.0*r*r + l*l) }" ixy="0" ixz="0"
+                iyy="${ (m/12.0) * (3.0*r*r + l*l) }" iyz="0"
+                izz="${ (m/12.0) * (3.0*r*r + l*l) }" />
+        </inertial>
+    </xacro:macro>
 </robot>

File: ros2_ws/src/red_cherrybot_description/urdf/mobile_base.xacro (robot description, xacro)
@@ -27,4 +27,5 @@
             <material name="bright_white"/>
       </visual>
+      <xacro:wheel_inertia m="2.0" r="${wheel_radius}" l="${wheel_length}" o_xyz="0 0 0" o_rpy="${pi/2} 0 0"/>
     </link>
   </xacro:macro>

File: ros2_ws/src/red_cherrybot_description/urdf/model.urdf.xacro (robot description, xacro)
@@ -3,4 +3,3 @@
 <xacro:include filename="common_properties.xacro"/>
 <xacro:include filename="mobile_base.xacro"/>
-<!-- Method to use custom meshes designed in CAD Softwares: Create a meshes folder in the pkg, install the folder in CMakeLists.txt and then reference them in the URDF file. Use the mesh include filename syntax. Including the custom mesh in the URDF here is not difficult, but designing it is the actual hard part. We also need to Scale Down/Up frequently in urdf as original STL file of CAD is bigger/smaller.-->
 </robot>

Commit message: Feat: add caster_wheel_inertia macro for calculating caster wheel inertial properties and integrate it into mobile base

File: ros2_ws/src/red_cherrybot_description/urdf/common_properties.xacro (robot description, xacro)
@@ -30,3 +30,13 @@
         </inertial>
     </xacro:macro>
+    <xacro:macro name="caster_wheel_inertia" params="m r o_xyz o_rpy">
+        <inertial>
+            <mass value="${m}"/>
+            <origin xyz="${o_xyz}" rpy="${o_rpy}"/>
+            <inertia
+                ixx="${ (2.0/5.0) * m * r * r }" ixy="0" ixz="0"
+                iyy="${ (2.0/5.0) * m * r * r }" iyz="0"
+                izz="${ (2.0/5.0) * m * r * r }" />
+        </inertial>
+    </xacro:macro>
 </robot>

File: ros2_ws/src/red_cherrybot_description/urdf/mobile_base.xacro (robot description, xacro)
@@ -40,4 +40,5 @@
       <material name="bright_white"/>
     </visual>
+    <xacro:caster_wheel_inertia m="1.0" r="${wheel_radius/2.0}" o_xyz="0 0 0" o_rpy="0 0 0"/>
   </link>
   <link name="base_footprint_link">

Commit message: Feat: rename inertia macros for wheels and caster wheels to improve clarity and consistency

File: ros2_ws/src/red_cherrybot_description/urdf/common_properties.xacro (robot description, xacro)
@@ -20,5 +20,5 @@
         </inertial>
     </xacro:macro>
-    <xacro:macro name="wheel_inertia" params="m r l o_xyz o_rpy">
+    <xacro:macro name="cylinder_inertia" params="m r l o_xyz o_rpy">
         <inertial>
             <mass value="${m}"/>
@@ -27,8 +27,8 @@
                 ixx="${ (m/12.0) * (3.0*r*r + l*l) }" ixy="0" ixz="0"
                 iyy="${ (m/12.0) * (3.0*r*r + l*l) }" iyz="0"
-                izz="${ (m/12.0) * (3.0*r*r + l*l) }" />
+                izz="${ (m/2.0) * (r*r) }" />
         </inertial>
     </xacro:macro>
-    <xacro:macro name="caster_wheel_inertia" params="m r o_xyz o_rpy">
+    <xacro:macro name="sphere_inertia" params="m r o_xyz o_rpy">
         <inertial>
             <mass value="${m}"/>

File: ros2_ws/src/red_cherrybot_description/urdf/mobile_base.xacro (robot description, xacro)
@@ -27,5 +27,5 @@
             <material name="bright_white"/>
       </visual>
-      <xacro:wheel_inertia m="2.0" r="${wheel_radius}" l="${wheel_length}" o_xyz="0 0 0" o_rpy="${pi/2} 0 0"/>
+      <xacro:cylinder_inertia m="2.0" r="${wheel_radius}" l="${wheel_length}" o_xyz="0 0 0" o_rpy="${pi/2} 0 0"/>
     </link>
   </xacro:macro>
@@ -40,5 +40,5 @@
       <material name="bright_white"/>
     </visual>
-    <xacro:caster_wheel_inertia m="1.0" r="${wheel_radius/2.0}" o_xyz="0 0 0" o_rpy="0 0 0"/>
+    <xacro:sphere_inertia m="1.0" r="${wheel_radius/2.0}" o_xyz="0 0 0" o_rpy="0 0 0"/>
   </link>
   <link name="base_footprint_link">

Commit message: Add depot warehouse world and setup guide for Gazebo integration
- Created a new SDF world file `depot_warehouse.world` that includes a ground plane and a sun light source, along with the custom Depot model.
- Added a comprehensive setup guide `world_setup_guide.md` detailing the integration of the Depot model into the ROS 2 simulation, addressing previous loading issues, and providing instructions for proper model and world configuration.

File: ros2_ws/src/red_cherrybot_description/urdf/common_properties.xacro (robot description, xacro)
@@ -1,12 +1,10 @@
 <?xml version="1.0"?>
 <robot xmlns:xacro="http://www.ros.org/wiki/xacro">
-    <!-- Vibrant & Metallic Material Palette -->
-    <material name="cherry_light_red">
-        <!-- Bright, vibrant cherry red with high saturation -->
-        <color rgba="0.85 0.09 0.21 1.0" />
+    <!-- Gazebo-friendly material palette -->
+    <material name="robot_blue">
+        <color rgba="0.03 0.24 0.75 1.0" />
     </material>
-    <material name="bright_white">
-        <!-- Bright White finish -->
-        <color rgba="1 1 1 1.0"/>
+    <material name="wheel_blue">
+        <color rgba="0.015 0.06 0.18 1.0"/>
     </material>
     <xacro:macro name="box_inertia" params="m x y z o_xyz o_rpy">

File: ros2_ws/src/red_cherrybot_description/urdf/mobile_base.xacro (robot description, xacro)
@@ -12,5 +12,5 @@
       </geometry>
       <origin xyz="0 0 ${base_height/2.0}" rpy="0 0 0"/>
-      <material name="cherry_light_red"/>
+      <material name="robot_blue"/>
     </visual>
     <collision>
@@ -31,5 +31,5 @@
             </geometry>
             <origin xyz="0 0 0" rpy="${pi/2} 0 0"/>
-            <material name="bright_white"/>
+            <material name="wheel_blue"/>
       </visual>
       <collision>
@@ -52,5 +52,5 @@
       </geometry>
       <origin xyz="0 0 0" rpy="0 0 0"/>
-      <material name="bright_white"/>
+      <material name="wheel_blue"/>
     </visual>
     <collision>

Commit message: Camera Link Added at proper position and with proper orientation - No Plugin Setup yet.

File: ros2_ws/src/red_cherrybot_description/urdf/common_properties.xacro (robot description, xacro)
@@ -7,4 +7,7 @@
     <material name="wheel_blue">
         <color rgba="0.015 0.06 0.18 1.0"/>
+    </material>
+    <material name="camera_yellow">
+        <color rgba="0.9 0.9 0.0 1.0"/>
     </material>
     <xacro:macro name="box_inertia" params="m x y z o_xyz o_rpy">

File: ros2_ws/src/red_cherrybot_description/urdf/model.urdf.xacro (robot description, xacro)
@@ -4,3 +4,4 @@
 <xacro:include filename="mobile_base.xacro"/>
 <xacro:include filename="mobile_base_gazebo.xacro"/>
+<xacro:include filename="camera.xacro"/>
 </robot>

Commit message: Add arm.xacro file and update model.urdf.xacro to include arm properties and link

File: ros2_ws/src/red_cherrybot_description/urdf/common_properties.xacro (robot description, xacro)
@@ -10,4 +10,10 @@
     <material name="camera_yellow">
         <color rgba="0.9 0.9 0.0 1.0"/>
+    </material>
+    <material name="base_orange">
+        <color rgba="0.9 0.5 0.0 1.0"/>
+    </material>
+    <material name="golden_yellow">
+        <color rgba="1.0 0.84 0.0 1.0"/>
     </material>
     <xacro:macro name="box_inertia" params="m x y z o_xyz o_rpy">

File: ros2_ws/src/red_cherrybot_description/urdf/model.urdf.xacro (robot description, xacro)
@@ -5,3 +5,4 @@
 <xacro:include filename="mobile_base_gazebo.xacro"/>
 <xacro:include filename="camera.xacro"/>
+<xacro:include filename="arm.xacro"/>
 </robot>
