Commit message: Added forearm Link and fixed some errors of URDF Rendering.

File: ros2_ws/src/red_cherrybot_description/urdf/arm.xacro (robot description, xacro)
@@ -1,8 +1,8 @@
 <?xml version="1.0"?>
 <robot name="Red_Cherry_Bot" xmlns:xacro="http://www.ros.org/wiki/xacro">
-    <xacro:property name="base_length" value="0.1"/>
-    <xacro:property name="base_width" value="0.1"/>
-    <xacro:property name="base_height" value="0.04"/> <!-- height in doc was 0.02 or 0.01-->
-    <xacro:property name="base_mass" value="0.5"/>
+    <xacro:property name="arm_base_length" value="0.1"/>
+    <xacro:property name="arm_base_width" value="0.1"/>
+    <xacro:property name="arm_base_height" value="0.04"/>
+    <xacro:property name="arm_base_mass" value="0.5"/>
     <xacro:property name="arm_radius" value="0.02"/>
     <xacro:property name="arm_height" value="0.3"/>
@@ -12,16 +12,32 @@
         <visual>
             <geometry>
-                <box size="${base_length} ${base_width} ${base_height}"/>
+                <box size="${arm_base_length} ${arm_base_width} ${arm_base_height}"/>
             </geometry>
-            <origin xyz="0 0 0" rpy="0 0 0"/>
+            <origin xyz="0 0 ${arm_base_height/2.0}" rpy="0 0 0"/>
             <material name="base_orange"/>
         </visual>
         <collision>
             <geometry>
-                <box size="${base_length} ${base_width} ${base_height}"/>
+                <box size="${arm_base_length} ${arm_base_width} ${arm_base_height}"/>
             </geometry>
-            <origin xyz="0 0 0" rpy="0 0 0"/>
+            <origin xyz="0 0 ${arm_base_height/2.0}" rpy="0 0 0"/>
         </collision>
-        <xacro:box_inertia m="${base_mass}" x="${base_length}" y="${base_width}" z="${base_height}" o_xyz="0 0 0" o_rpy="0 0 0"/>
+        <xacro:box_inertia m="${arm_base_mass}" x="${arm_base_length}" y="${arm_base_width}" z="${arm_base_height}" o_xyz="0 0 ${arm_base_height/2.0}" o_rpy="0 0 0"/>
+    </link>
+    <link name="forearm_link">
+        <visual>
+            <geometry>
+                <cylinder radius="${arm_radius}" length="${arm_height}"/>
+            </geometry>
+            <origin xyz="0 0 ${arm_height/2.0}" rpy="0 0 0"/>
+            <material name="golden_yellow"/>
+        </visual>
+        <collision>
+            <geometry>
+                <cylinder radius="${arm_radius}" length="${arm_height}"/>
+            </geometry>
+            <origin xyz="0 0 ${arm_height/2.0}" rpy="0 0 0"/>
+        </collision>
+        <xacro:cylinder_inertia m="${arm_mass}" r="${arm_radius}" l="${arm_height}" o_xyz="0 0 ${arm_height/2.0}" o_rpy="0 0 0"/>
     </link>
     <!-- Joints -->
@@ -29,6 +45,12 @@
         <parent link="base_link"/>
         <child link="arm_base_link"/>
-        <origin xyz="0 0 0.4" rpy="0 0 0"/>
-        <!-- Warning, 0.4 is hardcoded here, should not have been ! I donno why ${base_height} is not working ! -->
+        <origin xyz="0 0 ${base_height}" rpy="0 0 0"/>
+    </joint>
+    <joint name="forearm_joint" type="revolute">
+        <parent link="arm_base_link"/>
+        <child link="forearm_link"/>
+        <origin xyz="0 0 ${arm_base_height}" rpy="0 0 0"/>
+        <axis xyz="0 1 0"/>
+        <limit effort="100" velocity="100" lower="0" upper="1.57"/>
     </joint>
 </robot>

Commit message: Add elbow link and joint to arm model; update materials for consistency

File: ros2_ws/src/red_cherrybot_description/urdf/arm.xacro (robot description, xacro)
@@ -41,4 +41,20 @@
         <xacro:cylinder_inertia m="${arm_mass}" r="${arm_radius}" l="${arm_height}" o_xyz="0 0 ${arm_height/2.0}" o_rpy="0 0 0"/>
     </link>
+    <link name="elbow_link">
+        <visual>
+            <geometry>
+                <cylinder radius="${arm_radius}" length="${arm_height}"/>
+            </geometry>
+            <origin xyz="0 0 ${arm_height/2.0}" rpy="0 0 0"/>
+            <material name="elbow_blue"/>
+        </visual>
+        <collision>
+            <geometry>
+                <cylinder radius="${arm_radius}" length="${arm_height}"/>
+            </geometry>
+            <origin xyz="0 0 ${arm_height/2.0}" rpy="0 0 0"/>
+        </collision>
+        <xacro:cylinder_inertia m="${arm_mass}" r="${arm_radius}" l="${arm_height}" o_xyz="0 0 ${arm_height/2.0}" o_rpy="0 0 0"/>
+    </link>
     <!-- Joints -->
     <joint name="arm_base_joint" type="fixed">
@@ -54,3 +70,10 @@
         <limit effort="100" velocity="100" lower="0" upper="1.57"/>
     </joint>
+    <joint name="elbow_joint" type="revolute">
+        <parent link="forearm_link"/>
+        <child link="elbow_link"/>
+        <origin xyz="0 0 ${arm_height}" rpy="0 0 0"/>
+        <axis xyz="0 1 0"/>
+        <limit effort="100" velocity="100" lower="0" upper="1.57"/>
+    </joint>
 </robot>

File: ros2_ws/src/red_cherrybot_description/urdf/common_properties.xacro (robot description, xacro)
@@ -2,9 +2,9 @@
 <robot xmlns:xacro="http://www.ros.org/wiki/xacro">
     <!-- Gazebo-friendly material palette -->
-    <material name="robot_blue">
-        <color rgba="0.03 0.24 0.75 1.0" />
+    <material name="base_cherry_red">
+        <color rgba="1.0 0.02 0.12 1.0" />
     </material>
-    <material name="wheel_blue">
-        <color rgba="0.015 0.06 0.18 1.0"/>
+    <material name="wheel_black">
+        <color rgba="0.0 0.0 0.0 1.0"/>
     </material>
     <material name="camera_yellow">
@@ -16,4 +16,10 @@
     <material name="golden_yellow">
         <color rgba="1.0 0.84 0.0 1.0"/>
+    </material>
+    <material name="red">
+        <color rgba="1.0 0.0 0.0 1.0"/>
+    </material>
+    <material name="elbow_blue">
+        <color rgba="0.0 0.2 1.0 1.0"/>
     </material>
     <xacro:macro name="box_inertia" params="m x y z o_xyz o_rpy">

File: ros2_ws/src/red_cherrybot_description/urdf/mobile_base.xacro (robot description, xacro)
@@ -12,5 +12,5 @@
       </geometry>
       <origin xyz="0 0 ${base_height/2.0}" rpy="0 0 0"/>
-      <material name="robot_blue"/>
+      <material name="base_cherry_red"/>
     </visual>
     <collision>
@@ -31,5 +31,5 @@
             </geometry>
             <origin xyz="0 0 0" rpy="${pi/2} 0 0"/>
-            <material name="wheel_blue"/>
+            <material name="wheel_black"/>
       </visual>
       <collision>
@@ -52,5 +52,5 @@
       </geometry>
       <origin xyz="0 0 0" rpy="0 0 0"/>
-      <material name="wheel_blue"/>
+      <material name="wheel_black"/>
     </visual>
     <collision>

Commit message: Add dynamics - (Friction and Damping) properties to arm joints for improved simulation behavior.

File: ros2_ws/src/red_cherrybot_description/urdf/arm.xacro (robot description, xacro)
@@ -69,4 +69,5 @@
         <axis xyz="0 1 0"/>
         <limit effort="100" velocity="100" lower="0" upper="1.57"/>
+        <dynamics damping="0.3" friction="0.3"/>
     </joint>
     <joint name="elbow_joint" type="revolute">
@@ -76,4 +77,5 @@
         <axis xyz="0 1 0"/>
         <limit effort="100" velocity="100" lower="0" upper="1.57"/>
+        <dynamics damping="0.3" friction="0.3"/>
     </joint>
 </robot>

Commit message: Everything fixed - Video made, Hope everything works now :) Fingers crossed !

File: ros2_ws/src/red_cherrybot_description/urdf/arm.xacro (robot description, xacro)
@@ -61,5 +61,5 @@
         <parent link="base_link"/>
         <child link="arm_base_link"/>
-        <origin xyz="0 0 ${base_height}" rpy="0 0 0"/>
+        <origin xyz="${base_length/4.0} 0 ${base_height}" rpy="0 0 0"/>
     </joint>
     <joint name="forearm_joint" type="revolute">

File: ros2_ws/src/red_cherrybot_description/urdf/arm_gazebo.xacro (robot description, xacro)
@@ -6,4 +6,5 @@
         <plugin filename="gz-sim-joint-position-controller-system" name="gz::sim::systems::JointPositionController">
             <joint_name>forearm_joint</joint_name>
+            <p_gain>3.0</p_gain>
         </plugin>
     </gazebo>
@@ -12,4 +13,5 @@
         <plugin filename="gz-sim-joint-position-controller-system" name="gz::sim::systems::JointPositionController">
             <joint_name>elbow_joint</joint_name>
+            <p_gain>3.0</p_gain>
         </plugin>
     </gazebo>
